File: kicad/SmartSwitch.kicad_pcb (KiCad board)
At the start: 2 copper layers, 48.3 x 83.8 mm, 34 parts, among them P1 DB, P2 MB, P3 P, P4 L, Q1 BC557, Q2 BT136, Q3 BC550, U1 MOC3042M, U2 MB133, U3 MB110

Commit message: +fix: clean code, naming +fix: pull down for reliable state after reset
Parts:
- added R2: 10k, Resistor_THT:R_Axial_DIN0207_L6.3mm_D2.5mm_P10.16mm_Horizontal, F.Cu at (59.7, 47.0)
- renumbered R9 to R10, R10 to R11, R2 to R3, R3 to R4, R4 to R5, R5 to R6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
Routing:
- net GND: track 81.3 -> 91.5 mm
