File: kicad/SmartSwitch.kicad_sch (KiCad schematic)
At the start: 34 parts, among them P1 DB, P2 MB, P3 P, P4 L, Q1 BC557, Q2 BT136, Q3 BC550, U1 MOC3042M, U2 MB133, U3 MB110

Commit message: +fix: clean code, naming +fix: pull down for reliable state after reset
Parts:
- added R2: 10k, Resistor_THT:R_Axial_DIN0207_L6.3mm_D2.5mm_P10.16mm_Horizontal, symbol Device:R_Small
- renumbered R9 to R10, R10 to R11, R2 to R3, R3 to R4, R4 to R5, R5 to R6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
Connections:
- net GND: now also R2.2
- net at H5.1, R4.2: now also R2.1
Other:
- moved on the sheet: H5, H6, R4
